Commit message: firmware test and IK test

File: src/manipulator_moveit/config/manipulator.ros2_control.xacro (robot description, xacro)
@@ -1,2 +1,58 @@
+<?xml version="1.0"?>
+<robot xmlns:xacro="http://www.ros.org/wiki/xacro">
+  <xacro:macro
+    name="manipulator_ros2_control"
+    params="name initial_positions_file hardware_plugin serial_port baud_rate timeout_ms control_mode">
+    <xacro:property
+      name="initial_positions"
+      value="${xacro.load_yaml(initial_positions_file)['initial_positions']}" />
+    <ros2_control name="${name}" type="system">
+      <hardware>
+        <!--
+          hardware_plugin 값에 따라 mock 또는 실제 ESP32 hardware interface를 선택한다.
+          mock:
+            mock_components/GenericSystem
+          real hardware:
+            manipulator_hardware/ManipulatorHardwareInterface
+        -->
+        <plugin>${hardware_plugin}</plugin>
+        <!-- ESP32 Serial 통신용 파라미터 -->
+        <param name="serial_port">${serial_port}</param>
+        <param name="baud_rate">${baud_rate}</param>
+        <param name="timeout_ms">${timeout_ms}</param>
+        <param name="control_mode">${control_mode}</param>
+      </hardware>
+      <joint name="joint1">
+        <command_interface name="position"/>
+        <state_interface name="position">
+          <param name="initial_value">${initial_positions['joint1']}</param>
+        </state_interface>
+        <state_interface name="velocity"/>
+      </joint>
+      <joint name="joint2">
+        <command_interface name="position"/>
+        <state_interface name="position">
+          <param name="initial_value">${initial_positions['joint2']}</param>
+        </state_interface>
+        <state_interface name="velocity"/>
+      </joint>
+      <joint name="joint3">
+        <command_interface name="position"/>
+        <state_interface name="position">
+          <param name="initial_value">${initial_positions['joint3']}</param>
+        </state_interface>
+        <state_interface name="velocity"/>
+      </joint>
+      <joint name="joint4">
+        <command_interface name="position"/>
+        <state_interface name="position">
+          <param name="initial_value">${initial_positions['joint4']}</param>
+        </state_interface>
+        <state_interface name="velocity"/>
+      </joint>
+    </ros2_control>
+  </xacro:macro>
+</robot>
+<!---
 <?xml version="1.0"?>
 <robot xmlns:xacro="http://www.ros.org/wiki/xacro">
@@ -5,7 +61,5 @@
         <ros2_control name="${name}" type="system">
             <hardware>
-                <!-- By default, set up controllers for simulation. This won't work on real hardware -->
                 <plugin>mock_components/GenericSystem</plugin>
-                <!--<plugin>manipulator_hardware/ManipulatorHardwareInterface</plugin>-->
             </hardware>
             <joint name="joint1">
@@ -40,2 +94,3 @@
     </xacro:macro>
 </robot>
+-->

File: src/manipulator_moveit/config/manipulator.urdf.xacro (robot description, xacro)
@@ -1,17 +1,65 @@
 <?xml version="1.0"?>
 <robot xmlns:xacro="http://www.ros.org/wiki/xacro" name="manipulator">
-  <!-- Initial joint positions -->
+  <!-- ========================================================= -->
+  <!-- Initial joint positions                                  -->
+  <!-- ========================================================= -->
+  <!-- open-loop PWM 서보에서는 실제 피드백이 없으므로 초기 상태 추정값으로 사용 -->
   <xacro:arg
     name="initial_positions_file"
     default="$(find manipulator_moveit)/config/initial_positions.yaml" />
-  <!-- Main robot model -->
+  <!-- ========================================================= -->
+  <!-- Hardware interface arguments                             -->
+  <!-- ========================================================= -->
+  <!-- mock에서 실제 ESP32 serial hardware interface로 전환하기 위한 설정 -->
+  <xacro:arg
+    name="hardware_plugin"
+    default="manipulator_hardware/ManipulatorHardwareInterface" />
+  <xacro:arg
+    name="serial_port"
+    default="/dev/ttyACM0" />
+  <xacro:arg
+    name="baud_rate"
+    default="115200" />
+  <xacro:arg
+    name="timeout_ms"
+    default="50" />
+  <xacro:arg
+    name="control_mode"
+    default="open_loop" />
+  <!-- ========================================================= -->
+  <!-- Main robot model                                         -->
+  <!-- ========================================================= -->
   <xacro:include
     filename="$(find manipulator)/description/capstone_manipulator.urdf.xacro" />
-  <!-- ros2_control configuration -->
+  <!-- ========================================================= -->
+  <!-- ros2_control configuration                               -->
+  <!-- ========================================================= -->
   <xacro:include
     filename="$(find manipulator_moveit)/config/manipulator.ros2_control.xacro" />
-  <!-- ros2_control fake/mock hardware instance -->
+  <!-- ========================================================= -->
+  <!-- ros2_control hardware instance                           -->
+  <!-- ========================================================= -->
+  <xacro:manipulator_ros2_control
+    name="manipulator_system"
+    initial_positions_file="$(arg initial_positions_file)"
+    hardware_plugin="$(arg hardware_plugin)"
+    serial_port="$(arg serial_port)"
+    baud_rate="$(arg baud_rate)"
+    timeout_ms="$(arg timeout_ms)"
+    control_mode="$(arg control_mode)" />
+</robot>
+<!--
+OLD manipulator.urdf.xacro backup
+<robot xmlns:xacro="http://www.ros.org/wiki/xacro" name="manipulator">
+  <xacro:arg
+    name="initial_positions_file"
+    default="$(find manipulator_moveit)/config/initial_positions.yaml" />
+  <xacro:include
+    filename="$(find manipulator)/description/capstone_manipulator.urdf.xacro" />
+  <xacro:include
+    filename="$(find manipulator_moveit)/config/manipulator.ros2_control.xacro" />
   <xacro:manipulator_ros2_control
     name="manipulator_system"
     initial_positions_file="$(arg initial_positions_file)" />
 </robot>
+-->
