Commit message: manipulator kinematics update

File: src/manipulator/description/capstone_manipulator.urdf.xacro (robot description, xacro)
@@ -1,9 +1,141 @@
-<?xml version="1.0" ?>
-<!-- =================================================================================== -->
-<!-- |    This document was autogenerated by xacro from capstone_manipulator.urdf.xacro | -->
-<!-- |    EDITING THIS FILE BY HAND IS NOT RECOMMENDED                                 | -->
-<!-- =================================================================================== -->
-<robot name="manipulator">
-  <!-- Optional materials for RViz -->
+<?xml version="1.0"?>
+<robot xmlns:xacro="http://www.ros.org/wiki/xacro" name="manipulator">
+  <!-- ========================================================= -->
+  <!-- 외부 Xacro include                                       -->
+  <!-- ========================================================= -->
+  <!-- RealSense D435 모델을 사용하기 위한 xacro include -->
+<xacro:include filename="/home/moonshot/Manipulator_only/src/realsense-ros/realsense2_description/urdf/_d435.urdf.xacro"/>
+  <!-- ========================================================= -->
+  <!-- 운동학 모델 정의                                         -->
+  <!-- ========================================================= -->
+  <!--
+    본 파일은 4축 직렬 다관절 로봇팔의 URDF Xacro 모델이다.
+    좌표계 및 단위:
+      - 길이 단위: meter [m]
+      - 회전 단위: radian [rad]
+      - +Z: 수직 상방
+      - +X: 로봇팔 전개 방향
+      - +Y: 오른손 좌표계 기준
+    운동학 체인:
+      link1 -> joint1 -> link2 -> joint2 -> link3
+            -> joint3 -> link4 -> joint4 -> link5
+            -> ee_fixed_joint -> ee_link
+            -> camera_joint -> camera_link
+    중요:
+      - mesh_xyz는 STL 형상의 표시 위치를 보정한다.
+      - joint*_origin_*는 실제 회전축 중심을 보정한다.
+      - 정지 상태 형상만 어긋나면 mesh_xyz를 수정한다.
+      - 회전할 때 축이 안 맞으면 joint origin을 수정한다.
+      - camera_link는 직접 box로 만들지 않고 realsense2_description의 D435 xacro를 사용한다.
+  -->
+  <!-- ========================================================= -->
+  <!-- 치수 변수 선언                                            -->
+  <!-- ========================================================= -->
+  <xacro:property name="link_w" value="0.050"/>
+  <xacro:property name="link_d" value="0.050"/>
+  <xacro:property name="base_h" value="0.048142"/>
+  <xacro:property name="joint1_to_joint2" value="0.068000"/>
+  <xacro:property name="joint2_to_joint3_z" value="0.262901"/>
+  <xacro:property name="joint2_to_joint3_x" value="0.030475"/>
+  <xacro:property name="joint3_to_joint4" value="0.346571"/>
+  <xacro:property name="wrist_link_len" value="0.080008"/>
+  <!-- 엔드이펙터 TCP 위치 -->
+  <xacro:property name="ee_offset_x" value="0.090008"/>
+  <xacro:property name="ee_offset_y" value="-0.033856"/>
+  <xacro:property name="ee_offset_z" value="0.019895"/>
+  <xacro:property name="ee_size" value="0.010"/>
+  <!-- D435 카메라 장착 위치 -->
+  <!-- 기존 camera_joint origin 값인 ${wrist_link_len / 2.0} 0 0.030을 변수화 -->
+  <xacro:property name="camera_origin_x" value="0.0"/>
+  <xacro:property name="camera_origin_y" value="0.000000"/>
+  <xacro:property name="camera_origin_z" value="0.035000"/>
+  <xacro:property name="camera_origin_roll" value="0.000000"/>
+  <xacro:property name="camera_origin_pitch" value="0.000000"/>
+  <xacro:property name="camera_origin_yaw" value="0.000000"/>
+  <!-- ========================================================= -->
+  <!-- 관절 회전축 중심 보정값                                   -->
+  <!-- ========================================================= -->
+  <!--
+    회전했을 때 STL의 구멍 중심과 실제 회전축이 어긋나면
+    아래 joint*_origin_* 값을 수정한다.
+    기준:
+      joint1 origin: link1 기준
+      joint2 origin: link2 기준
+      joint3 origin: link3 기준
+      joint4 origin: link4 기준
+  -->
+  <xacro:property name="joint1_origin_x" value="0.000000"/>
+  <xacro:property name="joint1_origin_y" value="0.000000"/>
+  <xacro:property name="joint1_origin_z" value="${base_h}"/>
+  <xacro:property name="joint2_origin_x" value="0.000000"/>
+  <xacro:property name="joint2_origin_y" value="0.000000"/>
+  <xacro:property name="joint2_origin_z" value="${joint1_to_joint2}"/>
+  <xacro:property name="joint3_origin_x" value="${joint2_to_joint3_x}"/>
+  <xacro:property name="joint3_origin_y" value="0.000000"/>
+  <xacro:property name="joint3_origin_z" value="${joint2_to_joint3_z}"/>
+  <xacro:property name="joint4_origin_x" value="${joint3_to_joint4}"/>
+  <xacro:property name="joint4_origin_y" value="0.000000"/>
+  <xacro:property name="joint4_origin_z" value="0.000000"/>
+  <!-- ========================================================= -->
+  <!-- 관절 회전축 방향                                          -->
+  <!-- ========================================================= -->
+  <!--
+    회전 중심은 맞는데 회전 방향이 반대이면 axis 부호를 바꾼다.
+    예: 0 1 0 -> 0 -1 0
+  -->
+  <xacro:property name="joint1_axis" value="0 0 1"/>
+  <xacro:property name="joint2_axis" value="0 1 0"/>
+  <xacro:property name="joint3_axis" value="0 1 0"/>
+  <xacro:property name="joint4_axis" value="0 1 0"/>
+  <!-- ========================================================= -->
+  <!-- STL mesh 설정                                             -->
+  <!-- ========================================================= -->
+  <xacro:property name="mesh_scale" value="0.001 0.001 0.001"/>
+  <!-- STL 위치 보정값 -->
+  <xacro:property name="base_mesh_xyz" value="-0.022 0.0385 0.04"/>
+  <xacro:property name="base_mesh_rpy" value="0 0 0"/>
+  <xacro:property name="link1_mesh_xyz" value="-0.022 0.0385 -0.0028"/>
+  <xacro:property name="link1_mesh_rpy" value="0 0 0"/>
+  <xacro:property name="link2_mesh_xyz" value="-0.023 0.0385 -0.0705"/>
+  <xacro:property name="link2_mesh_rpy" value="0 0 0"/>
+  <xacro:property name="link3_mesh_xyz" value="-0.0538 0.0385 -0.3335"/>
+  <xacro:property name="link3_mesh_rpy" value="0 0 0"/>
+  <xacro:property name="link4_mesh_xyz" value="-0.43 0.0385 -0.334"/>
+  <xacro:property name="link4_mesh_rpy" value="0 0 0"/>
+  <!-- ========================================================= -->
+  <!-- 관절 제한값                                               -->
+  <!-- ========================================================= -->
+  <xacro:property name="joint1_lower" value="-3.14159265359"/>
+  <xacro:property name="joint1_upper" value="3.14159265359"/>
+  <xacro:property name="joint2_lower" value="-1.57"/>
+  <xacro:property name="joint2_upper" value="2.1"/>
+  <xacro:property name="joint3_lower" value="-1.57"/>
+  <xacro:property name="joint3_upper" value="1.57"/>
+  <xacro:property name="joint4_lower" value="-1.5"/>
+  <xacro:property name="joint4_upper" value="1.5"/>
+  <xacro:property name="joint_effort" value="0.1"/>
+  <xacro:property name="joint_velocity" value="4.8"/>
+  <!-- ========================================================= -->
+  <!-- 재사용 매크로                                             -->
+  <!-- ========================================================= -->
+  <xacro:macro name="mesh_visual" params="mesh_file xyz rpy material_name">
+    <visual>
+      <origin xyz="${xyz}" rpy="${rpy}"/>
+      <geometry>
+        <mesh filename="package://manipulator/model/${mesh_file}" scale="${mesh_scale}"/>
+      </geometry>
+      <material name="${material_name}"/>
+    </visual>
+  </xacro:macro>
+  <xacro:macro name="simple_inertial" params="xyz mass ixx iyy izz">
+    <inertial>
+      <origin xyz="${xyz}" rpy="0 0 0"/>
+      <mass value="${mass}"/>
+      <inertia ixx="${ixx}" ixy="0" ixz="0" iyy="${iyy}" iyz="0" izz="${izz}"/>
+    </inertial>
+  </xacro:macro>
+  <!-- ========================================================= -->
+  <!-- Materials                                                 -->
+  <!-- ========================================================= -->
   <material name="grey">
     <color rgba="0.2 0.2 0.2 1.0"/>
@@ -15,197 +147,190 @@
     <color rgba="0.6 0.1 0.1 1.0"/>
   </material>
-  <!-- =========================
-       link1 (base block on robot, bottom at z=0)
-       size: 0.05 x 0.05 x 0.05
-       ========================= -->
+  <!-- ========================================================= -->
+  <!-- link1: base block                                         -->
+  <!-- STL: base_link.stl                                        -->
+  <!-- ========================================================= -->
   <link name="link1">
-    <visual>
-      <origin rpy="0 0 0" xyz="0 0 0.025"/>
-      <geometry>
-        <box size="0.05 0.05 0.05"/>
-      </geometry>
-      <material name="dark_grey"/>
-    </visual>
-    <collision>
-      <origin rpy="0 0 0" xyz="0 0 0.025"/>
-      <geometry>
-        <box size="0.05 0.05 0.05"/>
-      </geometry>
-    </collision>
-    <inertial>
-      <origin rpy="0 0 0" xyz="0 0 0.025"/>
-      <mass value="1.0"/>
-      <inertia ixx="0.0004166667" ixy="0" ixz="0" iyy="0.0004166667" iyz="0" izz="0.0004166667"/>
-    </inertial>
-  </link>
-  <!-- joint1: base yaw (Z) -->
+    <xacro:mesh_visual
+      mesh_file="base_link.stl"
+      xyz="${base_mesh_xyz}"
+      rpy="${base_mesh_rpy}"
+      material_name="dark_grey"/>
+    <collision>
+      <origin xyz="0 0 ${base_h / 2.0}" rpy="0 0 0"/>
+      <geometry>
+        <box size="${link_w} ${link_d} ${base_h}"/>
+      </geometry>
+    </collision>
+    <xacro:simple_inertial
+      xyz="0 0 ${base_h / 2.0}"
+      mass="1.0"
+      ixx="0.0004166667"
+      iyy="0.0004166667"
+      izz="0.0004166667"/>
+  </link>
+  <!-- ========================================================= -->
+  <!-- joint1: base yaw                                          -->
+  <!-- ========================================================= -->
   <joint name="joint1" type="revolute">
     <parent link="link1"/>
     <child link="link2"/>
-    <origin rpy="0 0 0" xyz="0 0 0.05"/>
-    <axis xyz="0 0 1"/>
-    <limit effort="0.1" lower="-3.14159265359" upper="3.14159265359" velocity="4.8"/>
-  </joint>
-  <!-- =========================
-       link2 (vertical riser)
-       length: 0.12m, cross-section: 0.05 x 0.05
-       ========================= -->
+    <origin xyz="${joint1_origin_x} ${joint1_origin_y} ${joint1_origin_z}" rpy="0 0 0"/>
+    <axis xyz="${joint1_axis}"/>
+    <limit effort="${joint_effort}" lower="${joint1_lower}" upper="${joint1_upper}" velocity="${joint_velocity}"/>
+  </joint>
+  <!-- ========================================================= -->
+  <!-- link2: joint1-to-joint2 vertical link                     -->
+  <!-- STL: link_1.stl                                           -->
+  <!-- ========================================================= -->
   <link name="link2">
-    <visual>
-      <origin rpy="0 0 0" xyz="0 0 0.06"/>
-      <geometry>
-        <box size="0.05 0.05 0.12"/>
-      </geometry>
-      <material name="grey"/>
-    </visual>
-    <collision>
-      <origin rpy="0 0 0" xyz="0 0 0.06"/>
-      <geometry>
-        <box size="0.05 0.05 0.12"/>
-      </geometry>
-    </collision>
-    <inertial>
-      <origin rpy="0 0 0" xyz="0 0 0.06"/>
-      <mass value="0.8"/>
-      <inertia ixx="0.0019866667" ixy="0" ixz="0" iyy="0.0019866667" iyz="0" izz="0.0003333333"/>
-    </inertial>
-  </link>
-  <!-- joint2: shoulder pitch (Y) at top of link2 -->
+    <xacro:mesh_visual
+      mesh_file="link_1.stl"
+      xyz="${link1_mesh_xyz}"
+      rpy="${link1_mesh_rpy}"
+      material_name="grey"/>
+    <collision>
+      <origin xyz="0 0 ${joint1_to_joint2 / 2.0}" rpy="0 0 0"/>
+      <geometry>
+        <box size="${link_w} ${link_d} ${joint1_to_joint2}"/>
+      </geometry>
+    </collision>
+    <xacro:simple_inertial
+      xyz="0 0 ${joint1_to_joint2 / 2.0}"
+      mass="0.8"
+      ixx="0.00035"
+      iyy="0.00035"
+      izz="0.0003333333"/>
+  </link>
+  <!-- ========================================================= -->
+  <!-- joint2: shoulder pitch                                    -->
+  <!-- ========================================================= -->
   <joint name="joint2" type="revolute">
     <parent link="link2"/>
     <child link="link3"/>
-    <origin rpy="0 0 0" xyz="0 0 0.12"/>
-    <axis xyz="0 1 0"/>
-    <limit effort="0.1" lower="-3.14159265359" upper="0.785398" velocity="4.8"/>
-  </joint>
-  <!-- =========================
-       link3 (upper arm)
-       length: 0.30m along +X, cross-section: 0.05 x 0.05
-       ========================= -->
+    <origin xyz="${joint2_origin_x} ${joint2_origin_y} ${joint2_origin_z}" rpy="0 0 0"/>
+    <axis xyz="${joint2_axis}"/>
+    <limit effort="${joint_effort}" lower="${joint2_lower}" upper="${joint2_upper}" velocity="${joint_velocity}"/>
+  </joint>
+  <!-- ========================================================= -->
+  <!-- link3: joint2-to-joint3 bent/protruded link               -->
+  <!-- STL: link_2.stl                                           -->
+  <!-- ========================================================= -->
   <link name="link3">
-    <visual>
-      <origin rpy="0 0 0" xyz="0.15 0 0"/>
-      <geometry>
-        <box size="0.30 0.05 0.05"/>
-      </geometry>
-      <material name="grey"/>
-    </visual>
-    <collision>
-      <origin rpy="0 0 0" xyz="0.15 0 0"/>
-      <geometry>
-        <box size="0.30 0.05 0.05"/>
-      </geometry>
-    </collision>
-    <inertial>
-      <origin rpy="0 0 0" xyz="0.15 0 0"/>
-      <mass value="0.6"/>
-      <inertia ixx="0.0002500000" ixy="0" ixz="0" iyy="0.0046250000" iyz="0" izz="0.0046250000"/>
-    </inertial>
-  </link>
-  <!-- joint3: elbow pitch (Y) at end of link3 -->
+    <xacro:mesh_visual
+      mesh_file="link_2.stl"
+      xyz="${link2_mesh_xyz}"
+      rpy="${link2_mesh_rpy}"
+      material_name="grey"/>
+    <collision>
+      <origin xyz="0 0 ${joint2_to_joint3_z / 2.0}" rpy="0 0 0"/>
+      <geometry>
+        <box size="${link_w} ${link_d} ${joint2_to_joint3_z}"/>
+      </geometry>
+    </collision>
+    <collision>
+      <origin xyz="${joint2_to_joint3_x / 2.0} 0 ${joint2_to_joint3_z}" rpy="0 0 0"/>
+      <geometry>
+        <box size="${joint2_to_joint3_x} ${link_d} ${link_w}"/>
+      </geometry>
+    </collision>
+    <xacro:simple_inertial
+      xyz="0 0 ${joint2_to_joint3_z / 2.0}"
+      mass="0.6"
+      ixx="0.0044"
+      iyy="0.0044"
+      izz="0.00025"/>
+  </link>
+  <!-- ========================================================= -->
+  <!-- joint3: elbow pitch                                       -->
+  <!-- ========================================================= -->
   <joint name="joint3" type="revolute">
     <parent link="link3"/>
     <child link="link4"/>
-    <origin rpy="0 0 0" xyz="0.30 0 0"/>
-    <axis xyz="0 1 0"/>
-    <limit effort="0.1" lower="0" upper="2.7" velocity="4.8"/>
-  </joint>
-  <!-- =========================
-       link4 (forearm)
-       length: 0.30m along +X
-       ========================= -->
+    <origin xyz="${joint3_origin_x} ${joint3_origin_y} ${joint3_origin_z}" rpy="0 0 0"/>
+    <axis xyz="${joint3_axis}"/>
+    <limit effort="${joint_effort}" lower="${joint3_lower}" upper="${joint3_upper}" velocity="${joint_velocity}"/>
+  </joint>
+  <!-- ========================================================= -->
+  <!-- link4: main horizontal arm                                -->
+  <!-- STL: link_3.stl                                           -->
+  <!-- ========================================================= -->
   <link name="link4">
-    <visual>
-      <origin rpy="0 0 0" xyz="0.15 0 0"/>
-      <geometry>
-        <box size="0.30 0.05 0.05"/>
-      </geometry>
-      <material name="grey"/>
-    </visual>
-    <collision>
-      <origin rpy="0 0 0" xyz="0.15 0 0"/>
-      <geometry>
-        <box size="0.30 0.05 0.05"/>
-      </geometry>
-    </collision>
-    <inertial>
-      <origin rpy="0 0 0" xyz="0.15 0 0"/>
-      <mass value="0.5"/>
-      <inertia ixx="0.0002083333" ixy="0" ixz="0" iyy="0.0038541667" iyz="0" izz="0.0038541667"/>
-    </inertial>
-  </link>
-  <!-- joint4: wrist pitch (Y) at end of link4 -->
+    <xacro:mesh_visual
+      mesh_file="link_3.stl"
+      xyz="${link3_mesh_xyz}"
+      rpy="${link3_mesh_rpy}"
+      material_name="grey"/>
+    <collision>
+      <origin xyz="${joint3_to_joint4 / 2.0} 0 0" rpy="0 0 0"/>
+      <geometry>
+        <box size="${joint3_to_joint4} ${link_d} ${link_w}"/>
+      </geometry>
+    </collision>
+    <xacro:simple_inertial
+      xyz="${joint3_to_joint4 / 2.0} 0 0"
+      mass="0.5"
+      ixx="0.0002083333"
+      iyy="0.0062"
+      izz="0.0062"/>
+  </link>
+  <!-- ========================================================= -->
+  <!-- joint4: wrist pitch                                       -->
+  <!-- ========================================================= -->
   <joint name="joint4" type="revolute">
     <parent link="link4"/>
     <child link="link5"/>
-    <origin rpy="0 0 0" xyz="0.30 0 0"/>
-    <axis xyz="0 1 0"/>
-    <limit effort="0.1" lower="-1.5" upper="1.5" velocity="4.8"/>
-  </joint>
+    <origin xyz="${joint4_origin_x} ${joint4_origin_y} ${joint4_origin_z}" rpy="0 0 0"/>
+    <axis xyz="${joint4_axis}"/>
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
File: src/realsense-ros/realsense2_description/urdf/_d435.urdf.xacro (robot description, xacro)
@@ -21,6 +21,4 @@
 <robot name="sensor_d435" xmlns:xacro="http://ros.org/wiki/xacro">
   <!-- Includes -->
-  <xacro:include filename="$(find realsense2_description)/urdf/_materials.urdf.xacro" />
-  <xacro:include filename="$(find realsense2_description)/urdf/_usb_plug.urdf.xacro" />
   <xacro:macro name="sensor_d435" params="parent *origin name:=camera use_nominal_extrinsics:=false add_plug:=false use_mesh:=true">
     <xacro:property name="M_PI" value="3.1415926535897931" />

Commit message: manipulator kinematics update

File: src/manipulator/description/capstone_manipulator.urdf.xacro (robot description, xacro)
@@ -34,14 +34,14 @@
   <xacro:property name="link_w" value="0.050"/>
   <xacro:property name="link_d" value="0.050"/>
-  <xacro:property name="base_h" value="0.048142"/>
-  <xacro:property name="joint1_to_joint2" value="0.068000"/>
-  <xacro:property name="joint2_to_joint3_z" value="0.262901"/>
-  <xacro:property name="joint2_to_joint3_x" value="0.030475"/>
-  <xacro:property name="joint3_to_joint4" value="0.346571"/>
-  <xacro:property name="wrist_link_len" value="0.080008"/>
+  <xacro:property name="base_h" value="0.088576"/>
+  <xacro:property name="joint1_to_joint2" value="0.058118"/>
+  <xacro:property name="joint2_to_joint3_z" value="0.263683"/>
+  <xacro:property name="joint2_to_joint3_x" value="0.031016"/>
+  <xacro:property name="joint3_to_joint4" value="0.346599"/>
+  <xacro:property name="wrist_link_len" value="0.090002"/>
   <!-- 엔드이펙터 TCP 위치 -->
-  <xacro:property name="ee_offset_x" value="0.090008"/>
-  <xacro:property name="ee_offset_y" value="-0.033856"/>
-  <xacro:property name="ee_offset_z" value="0.019895"/>
+  <xacro:property name="ee_offset_x" value="0.090002"/>
+  <xacro:property name="ee_offset_y" value="-0.034040"/>
+  <xacro:property name="ee_offset_z" value="0.019938"/>
   <xacro:property name="ee_size" value="0.010"/>
   <!-- D435 카메라 장착 위치 -->
@@ -93,11 +93,11 @@
   <xacro:property name="mesh_scale" value="0.001 0.001 0.001"/>
   <!-- STL 위치 보정값 -->
-  <xacro:property name="base_mesh_xyz" value="-0.022 0.0385 0.04"/>
+  <xacro:property name="base_mesh_xyz" value="-0.02 -0.1815 0.077"/>
   <xacro:property name="base_mesh_rpy" value="0 0 0"/>
-  <xacro:property name="link1_mesh_xyz" value="-0.022 0.0385 -0.0028"/>
+  <xacro:property name="link1_mesh_xyz" value="-0.022 0.0385 -0.012"/>
   <xacro:property name="link1_mesh_rpy" value="0 0 0"/>
-  <xacro:property name="link2_mesh_xyz" value="-0.023 0.0385 -0.0705"/>
+  <xacro:property name="link2_mesh_xyz" value="-0.022 0.0385 -0.0701"/>
   <xacro:property name="link2_mesh_rpy" value="0 0 0"/>
-  <xacro:property name="link3_mesh_xyz" value="-0.0538 0.0385 -0.3335"/>
+  <xacro:property name="link3_mesh_xyz" value="-0.053 0.0385 -0.3339"/>
   <xacro:property name="link3_mesh_rpy" value="0 0 0"/>
   <xacro:property name="link4_mesh_xyz" value="-0.43 0.0385 -0.334"/>

Commit message: mani kinematics update

File: src/manipulator/description/capstone_manipulator.urdf.xacro (robot description, xacro)
@@ -5,6 +5,5 @@
   <!-- ========================================================= -->
   <!-- RealSense D435 모델을 사용하기 위한 xacro include -->
-<xacro:include filename="/home/moonshot/Manipulator_only/src/realsense-ros/realsense2_description/urdf/_d435.urdf.xacro"/>
-  <!-- ========================================================= -->
+<xacro:include filename="$(find realsense2_description)/urdf/_d435.urdf.xacro"/>  <!-- ========================================================= -->
   <!-- 운동학 모델 정의                                         -->
   <!-- ========================================================= -->
@@ -112,6 +111,6 @@
   <xacro:property name="joint3_lower" value="-1.57"/>
   <xacro:property name="joint3_upper" value="1.57"/>
-  <xacro:property name="joint4_lower" value="-1.5"/>
-  <xacro:property name="joint4_upper" value="1.5"/>
+  <xacro:property name="joint4_lower" value="-0.5"/>
+  <xacro:property name="joint4_upper" value="0.7"/>
   <xacro:property name="joint_effort" value="0.1"/>
   <xacro:property name="joint_velocity" value="4.8"/>
