Commit message: kinematics update

File: src/manipulator/description/capstone_manipulator.urdf.xacro (robot description, xacro)
@@ -105,14 +105,12 @@
   <!-- 관절 제한값                                               -->
   <!-- ========================================================= -->
-  <xacro:property name="joint1_lower" value="-3.14159265359"/>
-  <xacro:property name="joint1_upper" value="3.14159265359"/>
-  <xacro:property name="joint2_lower" value="-1.57"/>
-  <xacro:property name="joint2_upper" value="2.1"/>
-  <xacro:property name="joint3_lower" value="-1.57"/>
-  <xacro:property name="joint3_upper" value="1.57"/>
-  <xacro:property name="joint4_lower" value="-0.5"/>
-  <xacro:property name="joint4_upper" value="0.7"/>
-  <xacro:property name="joint_effort" value="0.1"/>
-  <xacro:property name="joint_velocity" value="4.8"/>
+  <xacro:property name="joint1_lower" value="-3.14159"/>  <!-- theta1_min = -180 deg -->
+  <xacro:property name="joint1_upper" value="0.0"/>       <!-- theta1_max =    0 deg -->
+  <xacro:property name="joint2_lower" value="-1.57080"/>  <!-- theta2_min =  -90 deg -->
+  <xacro:property name="joint2_upper" value="2.00713"/>   <!-- theta2_max =  115 deg -->
+  <xacro:property name="joint3_lower" value="-1.57080"/>  <!-- theta3_min =  -90 deg -->
+  <xacro:property name="joint3_upper" value="1.30900"/>   <!-- theta3_max =   75 deg -->
+  <xacro:property name="joint4_lower" value="-0.47124"/>  <!-- theta4_min =  -27 deg -->
+  <xacro:property name="joint4_upper" value="1.30900"/>   <!-- theta4_max =   75 deg -->
   <!-- ========================================================= -->
   <!-- 재사용 매크로                                             -->

File: src/manipulator_moveit/config/manipulator.urdf.xacro (robot description, xacro)
@@ -17,5 +17,5 @@
   <xacro:arg
     name="serial_port"
-    default="/dev/ttyACM0" />
+    default="/dev/ttyUSB0" />
   <xacro:arg
     name="baud_rate"

Commit message: manager update

File: src/manipulator/description/capstone_manipulator.urdf.xacro (robot description, xacro)
@@ -111,5 +111,5 @@
   <xacro:property name="joint3_lower" value="-1.57080"/>  <!-- theta3_min =  -90 deg -->
   <xacro:property name="joint3_upper" value="1.30900"/>   <!-- theta3_max =   75 deg -->
-  <xacro:property name="joint4_lower" value="-0.47124"/>  <!-- theta4_min =  -27 deg -->
+  <xacro:property name="joint4_lower" value="-0.41888"/>  <!-- theta4_min =  -24 deg -->
   <xacro:property name="joint4_upper" value="1.30900"/>   <!-- theta4_max =   75 deg -->
   <!-- ========================================================= -->

Commit message: test

File: src/manipulator/description/capstone_manipulator.urdf.xacro (robot description, xacro)
@@ -110,7 +110,9 @@
   <xacro:property name="joint2_upper" value="2.00713"/>   <!-- theta2_max =  115 deg -->
   <xacro:property name="joint3_lower" value="-1.57080"/>  <!-- theta3_min =  -90 deg -->
-  <xacro:property name="joint3_upper" value="1.30900"/>   <!-- theta3_max =   75 deg -->
+  <xacro:property name="joint3_upper" value="1.30900"/>   <!-- theta3_max =   60 deg -->
   <xacro:property name="joint4_lower" value="-0.41888"/>  <!-- theta4_min =  -24 deg -->
-  <xacro:property name="joint4_upper" value="1.30900"/>   <!-- theta4_max =   75 deg -->
+  <xacro:property name="joint4_upper" value="1.22173"/>   <!-- theta4_max =   70 deg -->
+  <xacro:property name="joint_effort" value="0.1"/>
+  <xacro:property name="joint_velocity" value="4.8"/>
   <!-- ========================================================= -->
   <!-- 재사용 매크로                                             -->
